File: pcb/DCWiFiSwitch.kicad_sch (KiCad schematic)
At the start: 28 parts, among them J1 Out1, J2 Prog, J3 12-24V, Q2 AO3400A, U1 EL817, U2 ESP-12F, U3 TPS5430DDA

Commit message: wip
Parts:
- added D3: SS34, Diode_SMD:D_SMA, symbol Diode:SS34
- added D4: RED, Diode_SMD:D_0603_1608Metric, symbol Device:LED
- added R12: 2k7, Resistor_SMD:R_0603_1608Metric, symbol Device:R
- C1: value 4.7uF -> 10uF; Catalogue https://jlcpcb.com/partdetail/30577-1206B475K500NT/C29823 -> https://jlcpcb.com/partdetail/14236-CL31A106KBHNNNE/C13585; LCSC Part C29823 -> C13585
- C3, C4: value 47uF -> 22uF; footprint Capacitor_SMD:C_0805_2012Metric -> Capacitor_SMD:C_0603_1608Metric; Catalogue https://jlcpcb.com/partdetail/17464-CL21A476MQYNNNE/C16780 -> https://jlcpcb.com/partdetail/60514-CL10A226MQ8NRNC/C59461; LCSC Part C16780 -> C59461
- C5: value 1uF -> 100nF; footprint Capacitor_SMD:C_0805_2012Metric -> Capacitor_SMD:C_0603_1608Metric; Catalogue https://jlcpcb.com/partdetail/29074-CL21B105KBFNNNE/C28323 -> https://jlcpcb.com/partdetail/Yageo-CC0603KRX7R9BB104/C14663; LCSC Part C28323 -> C14663
- L1: value L -> 22uH; footprint (none) -> Inductor_SMD:L_Sunlord_SWPA4030S; Catalogue (none) -> https://jlcpcb.com/partdetail/Sunlord-SWPA4030S220MT/C83472; LCSC Part (none) -> C83472
- R2: value 1k -> 820R; Catalogue https://jlcpcb.com/partdetail/21904-0603WAF1001T5E/C21190 -> https://jlcpcb.com/partdetail/23980-0603WAF8200T5E/C23253; LCSC Part C21190 -> C23253
- R3: value 1k5 -> 2k7; Catalogue https://jlcpcb.com/partdetail/23570-0603WAF1501T5E/C22843 -> https://jlcpcb.com/partdetail/13814-0603WAF2701T5E/C13167; LCSC Part C22843 -> C13167
Connections:
- net GND: now also D3.2 (A), D4.1 (K); no longer R2.2
- net VCC: now also D3.1 (K)
- net at Q2.1 (G), R2.1, R3.2: now also R12.2
- net at R3.1, U1.3: now also R12.1
- new net: D4.2 (A), R2.2
- no-connect marks 1 -> 8
Other:
- moved on the sheet: C1, C2, C3, D2, L1, R1, R10, R11, R8, R9, U1, U3

Commit message: ready for pcb
Parts:
- added D5: SS34, Diode_SMD:D_SMA, symbol Diode:SS34
- added D6: RED, Diode_SMD:D_0603_1608Metric, symbol Device:LED
- added F3: Fuse, Fuse:Fuse_1206_3216Metric, symbol Device:Fuse
- added J3: Out1, TerminalBlock:TerminalBlock_bornier-2_P5.08mm, symbol Connector_Generic:Conn_01x02
- added Q2: AO3400A, Package_TO_SOT_SMD:SOT-23, symbol Transistor_FET:AO3400A
- added R13: 120R, Resistor_SMD:R_0603_1608Metric, symbol Device:R
- added R14, R15: 2k7, Resistor_SMD:R_0603_1608Metric, symbol Device:R
- added R16: 820R, Resistor_SMD:R_0603_1608Metric, symbol Device:R
- added U4: EL817, Package_DIP:DIP-4_W7.62mm, symbol Isolator:EL817
- renumbered C2 to C1, C1 to C2, C5 to C4, C4 to C5, D3 to D1, D1 to D3, F2 to F1, F1 to F2, J3 to J1, J1 to J2, J2 to J4, Q2 to Q1, R11 to R1, R12 to R10, R3 to R11, R2 to R12, R8 to R2, R9 to R3, R10 to R4, R7 to R5, R5 to R6, R6 to R7, R4 to R8, R1 to R9, U3 to U1, U1 to U3
Connections:
- net CTRL1: now also U2.19 (GPIO4)
- net GND: now also D6.1 (K), Q2.2 (S), U4.2
- net VCC: now also F3.1
- net CTRL2: now reaches U2.20 (GPIO5)
- net CTRL2: now also R13.2
- new net: R13.1, U4.1
- new net: R14.1, R15.1, U4.3
- new net: D5.1 (K), F3.2, J3.1 (Pin_1), U4.4
- new net: Q2.1 (G), R14.2, R15.2, R16.1
- new net: D6.2 (A), R16.2
- new net: D5.2 (A), J3.2 (Pin_2), Q2.3 (D)
- no-connect marks 8 -> 13
Other:
- moved on the sheet: C1, C2, C3, C4, C5, D1, D2, D3, D4, F1, F2, J1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

Commit message: board rc1
Parts:
- removed J1: 12-24V, TerminalBlock:TerminalBlock_bornier-2_P5.08mm, symbol Connector_Generic:Conn_01x02
- removed J2, J3: Out1, TerminalBlock:TerminalBlock_bornier-2_P5.08mm, symbol Connector_Generic:Conn_01x02
- added C3: 100nF, Capacitor_SMD:C_0603_1608Metric, symbol Device:C
- added H1, H2, H3, H4: MH, MountingHole:MountingHole_3.2mm_M3_ISO7380_Pad, symbol Mechanical:MountingHole_Pad
- added J1: Screw_Terminal_01x06, TerminalBlock_Phoenix:TerminalBlock_Phoenix_MKDS-1,5-6-5.08_1x06_P5.08mm_Horizontal, symbol Connector:Screw_Terminal_01x06
- U3, U4: footprint Package_DIP:DIP-4_W7.62mm -> Package_DIP:SMDIP-4_W9.53mm
- renumbered C3 to C4, C4 to C5, C5 to C6
Connections:
- net CTRL1: now also U2.6 (GPIO12); no longer U2.19 (GPIO4)
- net CTRL2: now also U2.5 (GPIO14); no longer U2.20 (GPIO5)
- net EN: now also J4.4 (Pin_4); no longer J4.5 (Pin_5)
- net GND: now also C3.2, H1.1, H2.1, H3.1, H4.1, J1.5 (Pin_5)
- net NRST: now also J4.5 (Pin_5); no longer J4.4 (Pin_4)
- net OUT2_P: now reaches D5.1 (K), F3.2, U4.4
- net OUT2_P: now also J1.2 (Pin_2)
- net OUT1_P: now reaches D3.1 (K), F2.2, U3.4
- net OUT1_P: now also J1.4 (Pin_4)
- net OUT2_N: now reaches D5.2 (A), Q2.3 (D)
- net OUT2_N: now also J1.1 (Pin_1)
- net OUT1_N: now reaches D3.2 (A), Q1.3 (D)
- net OUT1_N: now also J1.3 (Pin_3)
- net PWR_INPUT: now reaches F1.1
- net PWR_INPUT: now also F2.1, F3.1, J1.6 (Pin_6)
- net VCC: no longer names the net of C2.1, D1.1 (K), F1.2, U1.7 (VIN)
- net VCC: now also C3.1; no longer F2.1, F3.1
Other:
- moved on the sheet: C1, C2, C4, D1, D2, D5, D6, F1, F3, L1, Q2, R1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

Commit message: board rc2
Parts:
- removed H3, H4: MH, MountingHole:MountingHole_3.2mm_M3_ISO7380_Pad, symbol Mechanical:MountingHole_Pad
- removed J4: Prog, Connector_PinHeader_2.54mm:PinHeader_1x05_P2.54mm_Vertical, symbol Connector_Generic:Conn_01x05
- added H1, H2: MH, MountingHole:MountingHole_3.2mm_M3_ISO7380, symbol Mechanical:MountingHole
- added J2: Conn_01x06, Connector_PinHeader_2.54mm:PinHeader_1x06_P2.54mm_Vertical, symbol Connector_Generic:Conn_01x06
- added R10, R5: 10k, Resistor_SMD:R_0603_1608Metric, symbol Device:R
- renumbered D3 to D1, D4 to D2, D5 to D3, D6 to D4, D1 to D5, D2 to D6, F2 to F1, F3 to F2, F1 to F3, H1 to H3, H2 to H4, R9 to R1, R1 to R11, R2 to R12, R3 to R13, R4 to R14, R5 to R15, R6 to R16, R7 to R17, R8 to R18, R10 to R2, R11 to R3, R12 to R4, R13 to R6, R14 to R7, R15 to R8, R16 to R9, U3 to U1, U4 to U2, U1 to U3, U2 to U4
Connections:
- net EN: now also J2.5 (Pin_5)
- net GND: now also J2.2 (Pin_2), R10.1, R5.1
- net NRST: now also J2.6 (Pin_6)
- net RXD: now also J2.4 (Pin_4)
- net TXD: now also J2.3 (Pin_3)
- net at D2.2 (A), R4.2: now also R5.2
- net at D4.2 (A), R9.2: now also R10.2
- net ADC: now reaches U4.2 (ADC)
- net ADC: now also J2.1 (Pin_1)
- no-connect marks 13 -> 12
Other:
- moved on the sheet: D1, D2, D3, D4, F1, F2, Q1, Q2, R1, R2, R3, R4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

Commit message: board rc3
Parts:
- R14: renamed from R10; value 10k -> 5k6; Catalogue https://jlcpcb.com/partdetail/26547-0603WAF1002T5E/C25804 -> https://jlcpcb.com/partdetail/23916-0603WAF5601T5E/C23189; LCSC Part C25804 -> C23189
- R9: renamed from R5; value 10k -> 5k6; Catalogue https://jlcpcb.com/partdetail/26547-0603WAF1002T5E/C25804 -> https://jlcpcb.com/partdetail/23916-0603WAF5601T5E/C23189; LCSC Part C25804 -> C23189
- renumbered D5 to D1, D6 to D2, D1 to D3, D2 to D4, D3 to D5, D4 to D6, F3 to F1, F1 to F2, F2 to F3, R11 to R1, R6 to R10, R7 to R11, R8 to R12, R9 to R13, R12 to R2, R13 to R3, R14 to R4, R1 to R5, R2 to R6, R3 to R7, R4 to R8, U3 to U1, U1 to U2, U2 to U3
Changed lines of the file:
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@@
 		(dnp no)
 		(fields_autoplaced yes)
-		(property "Reference" "R1"
+		(property "Reference" "R5"
 			(at 204.47 35.56 90)
 			(effects
@@
 			(project ""
 				(path "/2bcf36d7-c0ba-4c16-848a-400e98718055"
-					(reference "R1")
+					(reference "R5")
 					(unit 1)
 				)
@@
 		(on_board yes)
 		(dnp no)
-		(property "Reference" "D2"
+		(property "Reference" "D4"
 			(at 228.854 72.898 90)
 			(effects
@@
 			(project ""
 				(path "/2bcf36d7-c0ba-4c16-848a-400e98718055"
-					(reference "D2")
+					(reference "D4")
 					(unit 1)
 				)
@@
 		(dnp no)
 		(fields_autoplaced yes)
-		(property "Reference" "U2"
+		(property "Reference" "U3"
 			(at 218.44 109.22 0)
 			(effects
@@
 			(project "DCWiFiSwitch"
 				(path "/2bcf36d7-c0ba-4c16-848a-400e98718055"
-					(reference "U2")
+					(reference "U3")
 					(unit 1)
 				)
@@
 		(dnp no)
 		(fields_autoplaced yes)
-		(property "Reference" "R11"
+		(property "Reference" "R1"
 			(at 157.48 25.4 90)
 			(effects
@@
 			(project "DCWiFiSwitch"
 				(path "/2bcf36d7-c0ba-4c16-848a-400e98718055"
-					(reference "R11")
+					(reference "R1")
 					(unit 1)
 				)
@@
 		(dnp no)
 		(fields_autoplaced yes)
-		(property "Reference" "R9"
+		(property "Reference" "R13"
 			(at 236.22 135.8899 0)
 			(effects
@@
 			(project "DCWiFiSwitch"
 				(path "/2bcf36d7-c0ba-4c16-848a-400e98718055"
-					(reference "R9")
+					(reference "R13")
 					(unit 1)
 				)
@@
 		(dnp no)
 		(fields_autoplaced yes)
-		(property "Reference" "R4"
+		(property "Reference" "R8"
 			(at 236.22 62.2299 0)
 			(effects
@@
 			(project ""
 				(path "/2bcf36d7-c0ba-4c16-848a-400e98718055"
-					(reference "R4")
+					(reference "R8")
 					(unit 1)
 				)
@@
 		(dnp no)
 		(fields_autoplaced yes)
-		(property "Reference" "U1"
+		(property "Reference" "U2"
 			(at 218.44 35.56 0)
 			(effects
@@
 			(project ""
 				(path "/2bcf36d7-c0ba-4c16-848a-400e98718055"
-					(reference "U1")
+					(reference "U2")
 					(unit 1)
 				)
@@
 		(dnp no)
 		(fields_autoplaced yes)
-		(property "Reference" "R13"
+		(property "Reference" "R3"
 			(at 153.67 50.7999 0)
 			(effects
@@
 			(project "DCWiFiSwitch"
 				(path "/2bcf36d7-c0ba-4c16-848a-400e98718055"
-					(reference "R13")
+					(reference "R3")
 					(unit 1)
 				)
@@
 		(dnp no)
 		(fields_autoplaced yes)
-		(property "Reference" "U3"
+		(property "Reference" "U1"
 			(at 97.79 24.13 0)
 			(effects
@@
 			(project ""
 				(path "/2bcf36d7-c0ba-4c16-848a-400e98718055"
-					(reference "U3")
+					(reference "U1")
 					(unit 1)
 				)
@@
 		(dnp no)
 		(fields_autoplaced yes)
-		(property "Reference" "F1"
+		(property "Reference" "F2"
 			(at 245.11 35.5599 0)
 			(effects
@@
 			(project ""
 				(path "/2bcf36d7-c0ba-4c16-848a-400e98718055"
-					(reference "F1")
+					(reference "F2")
 					(unit 1)
 				)
@@
 		(dnp no)
 		(fields_autoplaced yes)
-		(property "Reference" "R12"
+		(property "Reference" "R2"
 			(at 153.67 36.8299 0)
 			(effects
@@
 			(project "DCWiFiSwitch"
 				(path "/2bcf36d7-c0ba-4c16-848a-400e98718055"
-					(reference "R12")
+					(reference "R2")
 					(unit 1)
 				)
@@
 		(on_board yes)
 		(dnp no)
-		(property "Reference" "R5"
+		(property "Reference" "R9"
 			(at 218.186 73.152 0)
 			(effects
@@
 			)
 		)
-		(property "Value" "10k"
+		(property "Value" "5k6"
 			(at 217.932 75.692 0)
 			(effects
@@
 			)
 		)
-		(property "Catalogue" "https://jlcpcb.com/partdetail/26547-0603WAF1002T5E/C25804"
+		(property "Catalogue" "https://jlcpcb.com/partdetail/23916-0603WAF5601T5E/C23189"
 			(at 223.52 73.66 0)
 			(effects
@@
 			)
 		)
-		(property "LCSC Part" "C25804"
+		(property "LCSC Part" "C23189"
 			(at 223.52 73.66 0)
 			(effects
@@
 			(project "DCWiFiSwitch"
 				(path "/2bcf36d7-c0ba-4c16-848a-400e98718055"
-					(reference "R5")
+					(reference "R9")
 					(unit 1)
 				)
@@
 		(dnp no)
 		(fields_autoplaced yes)
-		(property "Reference" "R3"
+		(property "Reference" "R7"
 			(at 236.22 52.0699 0)
 			(effects
@@
 			(project ""
 				(path "/2bcf36d7-c0ba-4c16-848a-400e98718055"
-					(reference "R3")
+					(reference "R7")
 					(unit 1)
 				)
@@
 		(dnp no)
 		(fields_autoplaced yes)
-		(property "Reference" "#PWR07"
+		(property "Reference" "#PWR08"
 			(at 95.25 55.88 0)
 			(effects
@@
 			(project "DCWiFiSwitch"
 				(path "/2bcf36d7-c0ba-4c16-848a-400e98718055"
-					(reference "#PWR07")
+					(reference "#PWR08")
 					(unit 1)
 				)
@@
 		(dnp no)
 		(fields_autoplaced yes)
-		(property "Reference" "D6"
+		(property "Reference" "D2"
 			(at 128.27 36.5124 90)
 			(effects
@@
 			(project "DCWiFiSwitch"
 				(path "/2bcf36d7-c0ba-4c16-848a-400e98718055"
-					(reference "D6")
+					(reference "D2")
 					(unit 1)
 				)
@@
 		(dnp no)
 		(fields_autoplaced yes)
-		(property "Reference" "F3"
+		(property "Reference" "F1"
 			(at 38.1 25.4 90)
 			(effects
@@
 			(project "DCWiFiSwitch"
 				(path "/2bcf36d7-c0ba-4c16-848a-400e98718055"
-					(reference "F3")
+					(reference "F1")
 					(unit 1)
 				)
@@
 		(on_board yes)
 		(dnp no)
-		(property "Reference" "R2"
+		(property "Reference" "R6"
 			(at 223.52 52.07 0)
 			(effects
@@
 			(project "DCWiFiSwitch"
 				(path "/2bcf36d7-c0ba-4c16-848a-400e98718055"
-					(reference "R2")
+					(reference "R6")
 					(unit 1)
 				)
@@
 		(dnp no)
 		(fields_autoplaced yes)
-		(property "Reference" "F2"
+		(property "Reference" "F3"
 			(at 245.11 109.2199 0)
 			(effects
@@
 			(project "DCWiFiSwitch"
 				(path "/2bcf36d7-c0ba-4c16-848a-400e98718055"
-					(reference "F2")
+					(reference "F3")
 					(unit 1)
 				)
@@
 		(dnp no)
 		(fields_autoplaced yes)
-		(property "Reference" "D5"
+		(property "Reference" "D1"
 			(at 49.53 36.5124 90)
 			(effects
@@
 			(project "DCWiFiSwitch"
 				(path "/2bcf36d7-c0ba-4c16-848a-400e98718055"
-					(reference "D5")
+					(reference "D1")
 					(unit 1)
 				)
@@
 		(on_board yes)
 		(dnp no)
-		(property "Reference" "R7"
+		(property "Reference" "R11"
 			(at 223.52 125.73 0)
 			(effects
@@
 			(project "DCWiFiSwitch"
 				(path "/2bcf36d7-c0ba-4c16-848a-400e98718055"
-					(reference "R7")
+					(reference "R11")
 					(unit 1)
 				)
@@
 		(on_board yes)
 		(dnp no)
-		(property "Reference" "D4"
+		(property "Reference" "D6"
 			(at 228.854 146.558 90)
 			(effects
@@
 			(project "DCWiFiSwitch"
 				(path "/2bcf36d7-c0ba-4c16-848a-400e98718055"
-					(reference "D4")
+					(reference "D6")
 					(unit 1)
 				)
@@
 		(dnp no)
 		(fields_autoplaced yes)
-		(property "Reference" "R8"
+		(property "Reference" "R12"
 			(at 236.22 125.7299 0)
 			(effects
@@
 			(project "DCWiFiSwitch"
 				(path "/2bcf36d7-c0ba-4c16-848a-400e98718055"
-					(reference "R8")
+					(reference "R12")
 					(unit 1)
 				)
@@
 		(dnp no)
 		(fields_autoplaced yes)
-		(property "Reference" "D3"
+		(property "Reference" "D5"
 			(at 245.11 119.0624 90)
 			(effects
@@
 			(project "DCWiFiSwitch"
 				(path "/2bcf36d7-c0ba-4c16-848a-400e98718055"
-					(reference "D3")
+					(reference "D5")
 					(unit 1)
 				)
@@
 		(dnp no)
 		(fields_autoplaced yes)
-		(property "Reference" "R14"
+		(property "Reference" "R4"
 			(at 153.67 58.4199 0)
 			(effects
@@
 			(project "DCWiFiSwitch"
 				(path "/2bcf36d7-c0ba-4c16-848a-400e98718055"
-					(reference "R14")
+					(reference "R4")
 					(unit 1)
 				)
@@
 		(dnp no)
 		(fields_autoplaced yes)
-		(property "Reference" "R6"
+		(property "Reference" "R10"
 			(at 204.47 109.22 90)
 			(effects
@@
 			(project "DCWiFiSwitch"
 				(path "/2bcf36d7-c0ba-4c16-848a-400e98718055"
-					(reference "R6")
+					(reference "R10")
 					(unit 1)
 				)
@@
 		(on_board yes)
 		(dnp no)
-		(property "Reference" "R10"
+		(property "Reference" "R14"
 			(at 218.186 146.812 0)
 			(effects
@@
 			)
 		)
-		(property "Value" "10k"
+		(property "Value" "5k6"
 			(at 217.932 149.352 0)
 			(effects
@@
 			)
 		)
-		(property "Catalogue" "https://jlcpcb.com/partdetail/26547-0603WAF1002T5E/C25804"
+		(property "Catalogue" "https://jlcpcb.com/partdetail/23916-0603WAF5601T5E/C23189"
 			(at 223.52 147.32 0)
 			(effects
@@
 			)
 		)
-		(property "LCSC Part" "C25804"
+		(property "LCSC Part" "C23189"
 			(at 223.52 147.32 0)
 			(effects
@@
 			(project "DCWiFiSwitch"
 				(path "/2bcf36d7-c0ba-4c16-848a-400e98718055"
-					(reference "R10")
+					(reference "R14")
 					(unit 1)
 				)
@@
 		(dnp no)
 		(fields_autoplaced yes)
-		(property "Reference" "#PWR08"
+		(property "Reference" "#PWR07"
 			(at 209.55 54.61 0)
 			(effects
@@
 			(project "DCWiFiSwitch"
 				(path "/2bcf36d7-c0ba-4c16-848a-400e98718055"
-					(reference "#PWR08")
+					(reference "#PWR07")
 					(unit 1)
 				)
@@
 		(dnp no)
 		(fields_autoplaced yes)
-		(property "Reference" "D1"
+		(property "Reference" "D3"
 			(at 245.11 45.4024 90)
 			(effects
@@
 			(project ""
 				(path "/2bcf36d7-c0ba-4c16-848a-400e98718055"
-					(reference "D1")
+					(reference "D3")
 					(unit 1)
 				)

Commit message: fixed gpio programmer, board rc4
Connections:
- net BOOT: now reaches R17.1, U4.18 (GPIO0)
- net BOOT: now also J2.5 (Pin_5)
- net EN: no longer names the net of R15.1, U4.3 (EN)
- net EN: no longer J2.5 (Pin_5)
Changed lines of the file:
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@@
 	(paper "A4")
 	(junction
-		(at 97.79 114.3)
-		(diameter 0)
-		(color 0 0 0 0)
-	)
-	(junction
 		(at 233.68 78.74)
 		(diameter 0)
@@
 	(junction
 		(at 123.19 31.75)
+		(diameter 0)
+		(color 0 0 0 0)
+	)
+	(junction
+		(at 140.97 109.22)
 		(diameter 0)
 		(color 0 0 0 0)
@@
 	(wire
 		(pts
-			(xy 95.25 114.3) (xy 97.79 114.3)
-		)
-		(stroke
-			(width 0)
-			(type default)
-		)
-	)
-	(wire
-		(pts
 			(xy 95.25 48.26) (xy 95.25 49.53)
 		)
@@
 		(pts
 			(xy 52.07 124.46) (xy 54.61 124.46)
+		)
+		(stroke
+			(width 0)
+			(type default)
+		)
+	)
+	(wire
+		(pts
+			(xy 140.97 109.22) (xy 142.24 109.22)
 		)
 		(stroke
@@
 		)
 	)
-	(global_label "EN"
+	(global_label "BOOT"
 		(shape input)
 		(at 54.61 121.92 0)
@@
 		)
 		(property "Intersheetrefs" "${INTERSHEET_REFS}"
-			(at 60.0747 121.92 0)
+			(at 62.4938 121.92 0)
 			(effects
 				(font
@@
 		)
 	)
-	(global_label "EN"
+	(global_label "BOOT"
 		(shape input)
-		(at 95.25 114.3 180)
+		(at 142.24 109.22 0)
 		(fields_autoplaced yes)
 		(effects
@@
 				(size 1.27 1.27)
 			)
-			(justify right)
+			(justify left)
 		)
 		(property "Intersheetrefs" "${INTERSHEET_REFS}"
-			(at 89.7853 114.3 0)
+			(at 150.1238 109.22 0)
 			(effects
 				(font
 					(size 1.27 1.27)
 				)
-				(justify right)
+				(justify left)
 				(hide yes)
 			)

Commit message: added more silkscreen help and a push button, rc5
Parts:
- added SW1: SW1_BOOT, Button_Switch_SMD:SW_Push_1P1T_XKB_TS-1187A, symbol Switch:SW_Push
Connections:
- net BOOT: now also SW1.1
- net GND: now also SW1.2
Changed lines of the file:
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@@
 	)
 	(junction
+		(at 152.4 109.22)
+		(diameter 0)
+		(color 0 0 0 0)
+	)
+	(junction
 		(at 242.57 125.73)
 		(diameter 0)
@@
 	(wire
 		(pts
+			(xy 152.4 109.22) (xy 152.4 110.49)
+		)
+		(stroke
+			(width 0)
+			(type default)
+		)
+	)
+	(wire
+		(pts
 			(xy 242.57 114.3) (xy 242.57 115.57)
 		)
@@
 	(wire
 		(pts
-			(xy 140.97 109.22) (xy 142.24 109.22)
+			(xy 140.97 109.22) (xy 152.4 109.22)
 		)
 		(stroke
@@
 	(wire
 		(pts
+			(xy 152.4 109.22) (xy 156.21 109.22)
+		)
+		(stroke
+			(width 0)
+			(type default)
+		)
+	)
+	(wire
+		(pts
 			(xy 125.73 31.75) (xy 125.73 34.29)
 		)
@@
 	(global_label "BOOT"
 		(shape input)
-		(at 142.24 109.22 0)
+		(at 156.21 109.22 0)
 		(fields_autoplaced yes)
 		(effects
@@
 		)
 		(property "Intersheetrefs" "${INTERSHEET_REFS}"
-			(at 150.1238 109.22 0)
+			(at 164.0938 109.22 0)
 			(effects
 				(font
@@
 	)
 	(symbol
+		(lib_id "Switch:SW_Push")
+		(at 152.4 115.57 270)
+		(unit 1)
+		(exclude_from_sim no)
+		(in_bom yes)
+		(on_board yes)
+		(dnp no)
+		(fields_autoplaced yes)
+		(property "Reference" "SW1"
+			(at 156.21 114.2999 90)
+			(effects
+				(font
+					(size 1.27 1.27)
+				)
+				(justify left)
+			)
+		)
+		(property "Value" "SW1_BOOT"
+			(at 156.21 116.8399 90)
+			(effects
+				(font
+					(size 1.27 1.27)
+				)
+				(justify left)
+			)
+		)
+		(property "Footprint" "Button_Switch_SMD:SW_Push_1P1T_XKB_TS-1187A"
+			(at 157.48 115.57 0)
+			(effects
+				(font
+					(size 1.27 1.27)
+				)
+				(hide yes)
+			)
+		)
+		(property "Datasheet" "~"
+			(at 157.48 115.57 0)
+			(effects
+				(font
+					(size 1.27 1.27)
+				)
+				(hide yes)
+			)
+		)
+		(property "Description" "Push button switch, generic, two pins"
+			(at 152.4 115.57 0)
+			(effects
+				(font
+					(size 1.27 1.27)
+				)
+				(hide yes)
+			)
+		)
+		(property "LCSC Part" "C318884"
+			(at 152.4 115.57 0)
+			(effects
+				(font
+					(size 1.27 1.27)
+				)
+				(hide yes)
+			)
+		)
+		(property "Catalogue" "https://jlcpcb.com/partdetail/XkbConnection-TS_1187A_B_AB/C318884"
+			(at 152.4 115.57 0)
+			(effects
+				(font
+					(size 1.27 1.27)
+				)
+				(hide yes)
+			)
+		)
+		(pin "2"
+		)
+		(pin "1"
+		)
+		(instances
+			(project ""
+				(path "/2bcf36d7-c0ba-4c16-848a-400e98718055"
+					(reference "SW1")
+					(unit 1)
+				)
+			)
+		)
+	)
+	(symbol
 		(lib_id "Device:L")
 		(at 132.08 31.75 90)
@@
 					(unit 1)
 				)
+			)
+		)
+	)
+	(symbol
+		(lib_id "power:GND")
+		(at 152.4 120.65 0)
+		(unit 1)
+		(exclude_from_sim no)
+		(in_bom yes)
+		(on_board yes)
+		(dnp no)
+		(fields_autoplaced yes)
+		(property "Reference" "#PWR027"
+			(at 152.4 127 0)
+			(effects
+				(font
+					(size 1.27 1.27)
+				)
+				(hide yes)
+			)
+		)
+		(property "Value" "GND"
+			(at 152.4 125.73 0)
+			(effects
+				(font
+					(size 1.27 1.27)
+				)
+			)
+		)
+		(property "Footprint" ""
+			(at 152.4 120.65 0)
+			(effects
+				(font
+					(size 1.27 1.27)
+				)
+				(hide yes)
+			)
+		)
+		(property "Datasheet" ""
+			(at 152.4 120.65 0)
+			(effects
+				(font
+					(size 1.27 1.27)
+				)
+				(hide yes)
+			)
+		)
+		(property "Description" "Power symbol creates a global label with name \"GND\" , ground"
+			(at 152.4 120.65 0)
+			(effects
+				(font
+					(size 1.27 1.27)
+				)
+				(hide yes)
+			)
+		)
+		(pin "1"
+		)
+		(instances
+			(project "DCWiFiSwitch"
+				(path "/2bcf36d7-c0ba-4c16-848a-400e98718055"
+					(reference "#PWR027")
+					(unit 1)
+				)
