File: pcb/DCWiFiSwitch.kicad_sch (KiCad schematic)
At the start: 47 parts, among them J1 Screw_Terminal_01x06, J2 Conn_01x07, Q1 AO3400A, Q2 AO3400A, SW1 SW1_BOOT, U1 TPS5430DDA, U2 EL817, U3 EL817, U4 ESP-12F

Commit message: add adc resistor divider
Parts:
- added R19: 220k, Resistor_SMD:R_0603_1608Metric, symbol Device:R
- added R20: 100k, Resistor_SMD:R_0603_1608Metric, symbol Device:R
Connections:
- net ADC: now also R19.2; no longer U4.2 (ADC)
- net GND: now also R20.1
- new net: R19.1, R20.2, U4.2 (ADC)
